Commit message: restructured nodes into one velocity control and integration/pose estimate node for preliminary testing

File: winter_project/urdf/diffbot.urdf (robot description, URDF)
Before this commit: robot test_robot, 4 links, 3 joints
Links:
- removed link fwheel_attach
- added link chassis_link; visual box size=0.16 0.16 0.06
- link base_link: geometry visual cylinder length=0.016 radius=0.023
Joints:
- removed joint base_to_fattach
- removed joint base_to_lconnection
- removed joint base_to_rconnection
- added joint base_to_chassis: type fixed, parent base_link, child chassis_link, origin xyz=0 0 0 rpy=0 0 0.008
- added joint chassis_to_lconnection: type fixed, parent chassis_link, child lwheel, origin xyz=0 0.084 0.046 rpy=0 0 1.57075
- added joint chassis_to_rconnection: type fixed, parent chassis_link, child rwheel, origin xyz=0 -0.084 0.046 rpy=0 0 1.57075
